Commit message: Close the perception-to-motion loop and validate it in Gazebo
Add 3D obstacle localization, a clearance-aware action adapter and a
shared RL contract, then run the full pipeline under ROS 2 Jazzy +
Gazebo Harmonic for the first time and fix what that exposed.

Perception-to-motion pipeline:
- obstacle_localizer: back-project detections with CameraInfo, transform
  them to base_link with TF at the image time, keep persistent tracks
- action_adapter: potential_field / rl / nominal modes behind one safety
  layer (whole-body clearance filter, speed, workspace and joint limits)
- rl_contract / scene_config: one observation layout and task frame
  shared by training and ROS; ur_kinematics, avoidance_logic,
  obstacle_tracker, camera_geometry as ROS-free modules

Gazebo integration fixes:
- Dockerfile: expose the venv to /usr/bin/python3 (vision_node died with
  "No module named 'ultralytics'"), add SB3, cache the Fuel chair
- World: the chair enclosed the TCP at the initial pose; put a geometric
  box on the path and the chair beyond it; lower the ground plane so the
  floor surface is at z = 0
- URDF: roll the camera mount by pi (images were upside down); spawn in
  a well-conditioned pose instead of the singular default
- action_adapter: send position-only trajectory points (the JTC rejected
  every command with a non-zero final velocity); start and stop episodes
  explicitly on /task/start and /task/stop
- rl_policy_node: load PPO checkpoints regardless of the NumPy version
  (a NumPy 2 pickle silently produced zero actions)

Perception:
- Class-agnostic depth fallback: near depth regions YOLO did not explain
  become "unknown" detections, localized at the region centroid
- Add "bench" to the target classes; report inference time and age
- Localizer drops measurements below min_height_m (floor)

RL:
- ur5e_scene: shaped reward, obstacle-position jitter, and a collision
  distance aligned with the safety filter (the legacy reward made
  stopping in front of the obstacle a local optimum)
- Bundle models/ppo_ur5e_scene.zip (1.5M steps)

Evaluation (methodology step 7):
- metrics_node: per-episode safety, control, perception and localization
  metrics against config/scene_ground_truth.yaml
- dataset_capture + scripts/benchmark_yolo.py: auto-labelled Gazebo
  frames and a YOLO model comparison (never downloads weights)
- scripts: run_gazebo_episode.sh (with readiness check and retry),
  capture_dataset.sh, evaluate_kinematic.py, summarize_metrics.py
- motion_loop: optional waypoints parameter

File: urdf/ur_gz_camera.urdf.xacro (robot description, xacro)
@@ -67,6 +67,9 @@
     <parent link="tool0"/>
     <child link="camera_link"/>
-    <!-- Change this pose to match the real camera bracket. -->
-    <origin xyz="0 0 0.08" rpy="0 0 0"/>
+    <!-- Change this pose to match the real camera bracket.
+         Gazebo cameras look along +X of the link and use +Z as image "up".
+         With the flange pointing down, rpy="0 0 0" produced upside-down images
+         (YOLO missed the chair); the roll of pi keeps the image upright. -->
+    <origin xyz="0 0 0.08" rpy="3.14159265359 0 0"/>
   </joint>
   <!-- ROS REP-103 optical frame: z forward, x right, y down. -->
@@ -105,7 +108,11 @@
     </plugin>
   </gazebo>
+  <!-- Start in a well-conditioned pose (the first motion_loop waypoint). The
+       upstream default (arm straight up) is singular: action_adapter refuses to
+       start there, and with commands enabled it would hold that pose. -->
   <xacro:ur_ros2_control
     name="$(arg name)"
     tf_prefix="$(arg tf_prefix)"
-    transmission_hw_interface="$(arg transmission_hw_interface)"/>
+    transmission_hw_interface="$(arg transmission_hw_interface)"
+    initial_positions="${dict(shoulder_pan_joint=0.0,shoulder_lift_joint=-1.2,elbow_joint=1.4,wrist_1_joint=-1.7,wrist_2_joint=-1.57,wrist_3_joint=0.0)}"/>
 </robot>
